Commit message: baseline

File: src/cpmr_apb/urdf/blockrobot.urdf.xacro (robot description, xacro)
@@ -36,5 +36,5 @@
     <visual>
       <geometry>
-        <cylinder length="0.05" radius="0.10" />
+        <cylinder length="0.1" radius="0.10" />
       </geometry>
       <!-- <geometry>
@@ -45,5 +45,5 @@
     <collision>
       <geometry>
-        <cylinder length="0.05" radius="0.10" />
+        <cylinder length="0.1" radius="0.10" />
       </geometry>
     </collision>

Commit message: following done. Does not go to correct goal

File: src/cpmr_apb/urdf/blockrobot.urdf.xacro (robot description, xacro)
@@ -36,5 +36,5 @@
     <visual>
       <geometry>
-        <cylinder length="0.1" radius="0.10" />
+        <cylinder length="0.15" radius="0.10" />
       </geometry>
       <!-- <geometry>
